File: TopPlate/ContraTopPlate.kicad_pcb (KiCad board)
At the start: 2 copper layers, 230.6 x 76.2 mm, 6 parts, among them p1 Plate

Commit message: Update plate files to latest
Other:
- board text added: "Contra Ortholinear Keyboard by ai03"
- board text added: "Plate Revision 1.6"
- board text removed: "Contra Ortho Keyboard Kit"
- board text removed: "Designed by Cartel and ai03"
- board text removed: "Plate Revision 1.5"
Changed lines of the file:
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@@
-(kicad_pcb (version 4) (host pcbnew 4.0.7)
+(kicad_pcb (version 20171130) (host pcbnew "(5.0.0)")
   (general
-    (links 1)
-    (no_connects 1)
-    (area 31.75 62.3748 279.5792 150.812501)
     (thickness 1.6)
-    (drawings 5)
+    (drawings 4)
     (tracks 0)
     (zones 0)
@@
     (visible_elements 7FFFFFFF)
     (pcbplotparams
-      (layerselection 0x010f0_80000001)
+      (layerselection 0x010f0_ffffffff)
       (usegerberextensions true)
-      (usegerberattributes true)
+      (usegerberattributes false)
+      (usegerberadvancedattributes false)
+      (creategerberjobfile false)
       (excludeedgelayer true)
       (linewidth 0.100000)
@@
       (hpglpennumber 1)
       (hpglpenspeed 20)
-      (hpglpendiameter 15)
-      (hpglpenoverlay 2)
+      (hpglpendiameter 15.000000)
       (psnegative false)
       (psa4output false)
@@
       (plotinvisibletext false)
       (padsonsilk false)
-      (subtractmaskfromsilk false)
+      (subtractmaskfromsilk true)
       (outputformat 1)
       (mirror false)
       (drillshape 0)
       (scaleselection 1)
-      (outputdirectory Gerbers))
+      (outputdirectory "Gerbers"))
   )
   (net 0 "")
@@
     (arrow2b (pts (xy 35.8902 65.0748) (xy 37.016704 64.488379)))
   )
-  (gr_text "Plate Revision 1.5" (at 232.791 124.46) (layer B.Mask)
+  (gr_text "Plate Revision 1.6" (at 232.791 124.46) (layer B.Mask)
     (effects (font (size 1.5 1.5) (thickness 0.3)) (justify mirror))
   )
-  (gr_text "Designed by Cartel and ai03" (at 227.076 105.41) (layer B.Mask)
+  (gr_text "Contra Ortholinear Keyboard by ai03\n" (at 222.25 86.36) (layer B.Mask)
     (effects (font (size 1.5 1.5) (thickness 0.3)) (justify mirror))
   )
-  (gr_text "Contra Ortho Keyboard Kit\n" (at 228.6 86.36) (layer B.Mask)
-    (effects (font (size 1.5 1.5) (thickness 0.3)) (justify mirror))
-  )
